File: Electronics/ESP01 + DHT11/ESP8266-01-DHT11_V3.brd (EAGLE design)
At the start: 27.9 x 30.7 mm, 6 parts, among them J1 22-27-2031-03, J2 22-27-2021-02

Commit message: - Updated electronics
Parts:
- renumbered IC1 to AMS1117, J1 to SERIAL, J2 to VIN, JP1 to PROG, U$1 to ESP8266-01
Connections:
- net N$2 renamed RX
- net N$3 renamed TX
- net N$5 renamed VIN+
Other:
- board text added: "ThingSpeak sens V3"
- board text removed: "FIWARE Sensor V3"
Changed lines of the file:
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@@
 <dimension x1="0" y1="0.254" x2="0" y2="28.956" x3="-6.35" y3="14.605" layer="20"/>
 <dimension x1="1.016" y1="-0.762" x2="26.924" y2="-0.762" x3="13.97" y3="-6.096" layer="20"/>
-<text x="6.985" y="10.795" size="1.016" layer="16" rot="MR135">FIWARE Sensor V3</text>
+<text x="6.731" y="10.541" size="1.016" layer="16" rot="MR135">ThingSpeak sens V3</text>
 <text x="15.875" y="20.955" size="1.016" layer="16" rot="MR315">@mifulapirus</text>
 </plain>
@@
 </autorouter>
 <elements>
-<element name="U$1" library="esp8266modules" package="ESP-01" value="ESP-01" x="6.985" y="12.7">
+<element name="ESP8266-01" library="esp8266modules" package="ESP-01" value="ESP-01" x="6.985" y="12.7">
 <attribute name="DIMENSIONS" value="14.3 x 24.8 mm" x="28.575" y="0" size="1.778" layer="27" display="off"/>
 <attribute name="PITCH" value="0.1&quot; / 2.54 mm" x="28.575" y="0" size="1.778" layer="27" display="off"/>
 <attribute name="PINS" value="8" x="28.575" y="0" size="1.778" layer="27" display="off"/>
 </element>
-<element name="IC1" library="v-reg-2" package="SOT223" value="" x="6.985" y="20.32" rot="MR180"/>
-<element name="JP1" library="jumper" package="JP1" value="" x="17.145" y="24.13"/>
-<element name="J1" library="con-molex" package="6410-03" value="22-27-2031-03" x="23.495" y="15.24" rot="R90">
+<element name="AMS1117" library="v-reg-2" package="SOT223" value="" x="6.985" y="20.32" rot="MR180"/>
+<element name="PROG" library="jumper" package="JP1" value="" x="17.145" y="24.13"/>
+<element name="SERIAL" library="con-molex" package="6410-03" value="22-27-2031-03" x="23.495" y="15.24" rot="R90">
 <attribute name="OC_NEWARK" value="unknown" x="29.845" y="50.8" size="1.778" layer="27" rot="R90" display="off"/>
 <attribute name="MPN" value="" x="29.845" y="50.8" size="1.778" layer="27" rot="R90" display="off"/>
@@
 </element>
 <element name="U$2" library="DHT11" package="DHT11-PION." value="DHT11-PION." x="20.955" y="6.35"/>
-<element name="J2" library="con-molex" package="6410-02" value="22-27-2021-02" x="23.495" y="24.13" rot="R90">
+<element name="VIN" library="con-molex" package="6410-02" value="22-27-2021-02" x="23.495" y="24.13" rot="R90">
 <attribute name="OC_NEWARK" value="unknown" x="59.055" y="43.18" size="1.778" layer="27" rot="R90" display="off"/>
 <attribute name="MPN" value="" x="59.055" y="43.18" size="1.778" layer="27" rot="R90" display="off"/>
@@
 <signals>
 <signal name="GND">
-<contactref element="IC1" pad="1"/>
-<contactref element="U$1" pad="GND"/>
-<contactref element="JP1" pad="2"/>
-<contactref element="J1" pad="3"/>
-<contactref element="U$2" pad="GND"/>
-<contactref element="J2" pad="2"/>
+<contactref element="AMS1117" pad="1"/>
+<contactref element="ESP8266-01" pad="GND"/>
+<contactref element="PROG" pad="2"/>
+<contactref element="SERIAL" pad="3"/>
+<contactref element="VIN" pad="2"/>
 <polygon width="0.4064" layer="16" isolate="0.6096">
 <vertex x="0" y="29.21"/>
@@
 <vertex x="0" y="-0.508"/>
 </polygon>
+<contactref element="U$2" pad="GND"/>
 </signal>
 <signal name="+3V3">
-<contactref element="IC1" pad="2"/>
-<contactref element="U$1" pad="VCC"/>
-<contactref element="U$1" pad="CH_PD"/>
+<contactref element="AMS1117" pad="2"/>
+<contactref element="ESP8266-01" pad="VCC"/>
+<contactref element="ESP8266-01" pad="CH_PD"/>
 <contactref element="U$2" pad="VCC"/>
 <wire x1="10.78" y1="4.5225" x2="15.9525" y2="4.5225" width="1.016" layer="16"/>
@@
 <wire x1="4.445" y1="9.525" x2="6.985" y2="12.065" width="0.4064" layer="16"/>
 <wire x1="5.7" y1="4.5225" x2="5.7" y2="3.19" width="0.4064" layer="16"/>
-<wire x1="5.7" y1="3.19" x2="6.985" y2="1.905" width="0.4064" layer="16"/>
-<wire x1="6.985" y1="1.905" x2="9.525" y2="1.905" width="0.4064" layer="16"/>
-<wire x1="9.525" y1="1.905" x2="10.795" y2="3.175" width="0.4064" layer="16"/>
+<wire x1="5.7" y1="3.19" x2="6.731" y2="2.159" width="0.4064" layer="16"/>
+<wire x1="6.731" y1="2.159" x2="9.779" y2="2.159" width="0.4064" layer="16"/>
+<wire x1="9.779" y1="2.159" x2="10.795" y2="3.175" width="0.4064" layer="16"/>
 <wire x1="10.795" y1="3.175" x2="10.795" y2="4.5075" width="0.4064" layer="16"/>
 <wire x1="10.795" y1="4.5075" x2="10.78" y2="4.5225" width="0.4064" layer="16"/>
@@
 </signal>
 <signal name="N$1">
-<contactref element="U$1" pad="GPIO0"/>
-<contactref element="JP1" pad="1"/>
+<contactref element="ESP8266-01" pad="GPIO0"/>
+<contactref element="PROG" pad="1"/>
 <wire x1="8.24" y1="7.0625" x2="8.24" y2="8.875" width="0.8128" layer="16"/>
 <wire x1="8.24" y1="8.875" x2="17.145" y2="17.78" width="0.8128" layer="16"/>
 <wire x1="17.145" y1="17.78" x2="17.145" y2="22.86" width="0.8128" layer="16"/>
 </signal>
-<signal name="N$2">
-<contactref element="J1" pad="2"/>
-<contactref element="U$1" pad="RX"/>
+<signal name="RX">
+<contactref element="SERIAL" pad="2"/>
+<contactref element="ESP8266-01" pad="RX"/>
 <wire x1="10.78" y1="7.0625" x2="13.9205" y2="7.0625" width="1.016" layer="16"/>
 <wire x1="13.9205" y1="7.0625" x2="16.764" y2="9.906" width="1.016" layer="16"/>
@@
 <wire x1="19.558" y1="10.922" x2="19.558" y2="13.97" width="1.016" layer="16"/>
 </signal>
-<signal name="N$3">
-<contactref element="J1" pad="1"/>
-<contactref element="U$1" pad="TX"/>
+<signal name="TX">
+<contactref element="SERIAL" pad="1"/>
+<contactref element="ESP8266-01" pad="TX"/>
 <wire x1="3.16" y1="4.5225" x2="3.16" y2="3.825" width="0.4064" layer="16"/>
 <wire x1="3.16" y1="3.825" x2="5.715" y2="1.27" width="0.4064" layer="16"/>
@@
 </signal>
 <signal name="N$4">
-<contactref element="U$1" pad="GPIO2"/>
+<contactref element="ESP8266-01" pad="GPIO2"/>
 <contactref element="U$2" pad="DATA"/>
 <wire x1="5.7" y1="7.0625" x2="5.7" y2="7" width="0.4064" layer="16"/>
@@
 <wire x1="19.558" y1="6.7818" x2="19.685" y2="6.6548" width="0.4064" layer="16"/>
 </signal>
-<signal name="N$5">
-<contactref element="J2" pad="1"/>
-<contactref element="IC1" pad="3"/>
+<signal name="VIN+">
+<contactref element="VIN" pad="1"/>
+<contactref element="AMS1117" pad="3"/>
 <wire x1="9.2964" y1="23.4188" x2="11.3538" y2="23.4188" width="0.8128" layer="16"/>
 <wire x1="11.3538" y1="23.4188" x2="15.24" y2="27.305" width="0.8128" layer="16"/>
