File: Electronics/ESP01 + DHT11/ESP8266-01-DHT11_V3.sch (EAGLE design)
At the start: 6 parts, among them J1 22-27-2031-03, J2 22-27-2021-02

Commit message: - Updated electronics
Parts:
- removed J1: 22-27-2031-03, con-molex:22-27-2031-03
- added SERIAL: 22-27-2031-03, con-molex:22-27-2031-03
- renumbered IC1 to AMS1117, J2 to VIN, JP1 to PROG, U$1 to ESP8266-01
Connections:
- net N$5 renamed VIN+
- removed net N$2: ESP8266-01.RXD, J1-2.S
- removed net N$3: ESP8266-01.TXD, J1-1.S
- new net RX: ESP8266-01.RXD, SERIAL-2.S
- new net TX: ESP8266-01.TXD, SERIAL-1.S
- net GND: now also SERIAL-3.S; no longer J1-3.S
Other:
- note added: "@mifulapirus"
- note added: "Author: Angel Hernandez"
- note added: "www.tupperbot.com"
